File: hardware/MBUS reader surface mount.brd (EAGLE design)
At the start: 20.5 x 71.8 mm, 18 parts, among them Q1 BC847, Q2 BC847, T1 BC857CSMD

Commit message: through hole with connector blocks
Changed lines of the file:
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@@
 <wire x1="75.7428" y1="79.4428" x2="75.7428" y2="7.62" width="0" layer="20"/>
 <wire x1="75.7428" y1="7.62" x2="96.09" y2="7.62" width="0" layer="20"/>
-<wire x1="3" y1="79.9" x2="3" y2="79.4" width="0" layer="121"/>
 <wire x1="96" y1="72" x2="96" y2="52" width="0.2032" layer="121"/>
 <wire x1="96" y1="52" x2="96" y2="29" width="0.2032" layer="121"/>
